Commit message: fix: correct material 'black' name && correct mesh path (hokuyo_ust10.stl)

File: dingo/dingo_description/urdf/accessories/hokuyo_ust10.urdf.xacro (robot description, xacro)
@@ -54,5 +54,5 @@
         <geometry>
           <!-- Origin of this mesh is the base of the bracket. -->
-          <mesh filename="$(find dingo_description)/meshes/hokuyo_ust10.stl" />
+          <mesh filename="file://$(find dingo_description)/meshes/hokuyo_ust10.stl" />
         </geometry>
         <material name="dark_grey" />

File: dingo/dingo_description/urdf/dingo-d.urdf.xacro (robot description, xacro)
@@ -74,5 +74,5 @@
         <sphere radius="0.01"/>
       </geometry>
-      <material name="Black"/>
+      <material name="black"/>
     </visual>
     <collision>

File: dingo_simulator/dingo_gazebo/urdf/dingo-d.urdf.xacro (robot description, xacro)
@@ -74,5 +74,5 @@
         <sphere radius="0.01"/>
       </geometry>
-      <material name="Black"/>
+      <material name="black"/>
     </visual>
     <collision>
